Commit message: Updated with changes and fixes

File: catkin_ws/src/my_robot/urdf/my_robot.xacro (robot description, xacro)
@@ -22,5 +22,5 @@
       <origin xyz="0 0 0" rpy=" 0 0 0"/>
       <geometry>
-        <box size=".4 .2 .1"/>
+        <box size=".8 .4 .2"/>
       </geometry>
     </collision>
@@ -28,30 +28,30 @@
       <origin xyz="0 0 0" rpy=" 0 0 0"/>
       <geometry>
-        <box size=".4 .2 .1"/>
+        <box size=".8 .4 .2"/>
       </geometry>
-      <material name="blue"/>
+      <material name="black"/>
     </visual>
     <collision name='back_caster_collision'>
-      <origin xyz="-0.15 0 -0.05" rpy=" 0 0 0"/>
+      <origin xyz="-0.15 0 -0.1" rpy=" 0 0 0"/>
       <geometry>
-        <sphere radius="0.0499"/>
+        <sphere radius="0.099"/>
       </geometry>
     </collision>
     <visual name='back_caster_visual'>
-      <origin xyz="-0.15 0 -0.05" rpy=" 0 0 0"/>
+      <origin xyz="-0.15 0 -0.1" rpy=" 0 0 0"/>
       <geometry>
-        <sphere radius="0.05"/>
+        <sphere radius="0.1"/>
       </geometry>
     </visual>
     <collision name='front_caster_collision'>
-      <origin xyz="0.15 0 -0.05" rpy=" 0 0 0"/>
+      <origin xyz="0.15 0 -0.1" rpy=" 0 0 0"/>
       <geometry>
-        <sphere radius="0.0499"/>
+        <sphere radius="0.099"/>
       </geometry>
     </collision>
     <visual name='front_caster_visual'>
-      <origin xyz="0.15 0 -0.05" rpy=" 0 0 0"/>
+      <origin xyz="0.15 0 -0.1" rpy=" 0 0 0"/>
       <geometry>
-        <sphere radius="0.05"/>
+        <sphere radius="0.1"/>
       </geometry>
     </visual>
@@ -66,5 +66,5 @@
       <origin xyz="0 0 0" rpy="0 1.5707 1.5707" />
       <geometry>
-          <cylinder radius='0.1' length='0.05' />
+          <cylinder radius='0.2' length='0.05' />
       </geometry>
     </collision>
@@ -72,7 +72,7 @@
       <origin xyz="0 0 0" rpy="0 1.5707 1.5707" />
       <geometry>
-          <cylinder radius='0.1' length='0.05' />
+          <cylinder radius='0.2' length='0.05' />
       </geometry>
-      <material name="green"/>
+      <material name="blue"/>
     </visual>
   </link>
@@ -90,5 +90,5 @@
       <origin xyz="0 0 0" rpy="0 1.5707 1.5707" />
       <geometry>
-          <cylinder radius="0.1" length="0.05" />
+          <cylinder radius="0.2" length="0.05" />
       </geometry>
     </collision>
@@ -96,11 +96,11 @@
       <origin xyz="0 0 0" rpy="0 1.5707 1.5707" />
       <geometry>
-          <cylinder radius='0.1' length='0.05' />
+          <cylinder radius='0.2' length='0.05' />
       </geometry>
-      <material name="green"/>
+      <material name="blue"/>
     </visual>
   </link>
   <joint type="continuous" name="left_wheel_hinge">
-    <origin xyz="0 0.15 0" rpy="0 0 0"/>
+    <origin xyz="0 0.25 0" rpy="0 0 0"/>
     <child link="left_wheel"/>
     <parent link="chassis"/>
@@ -111,5 +111,5 @@
   </joint>
   <joint type="continuous" name="right_wheel_hinge">
-    <origin xyz="0 -0.15 0" rpy="0 0 0"/>
+    <origin xyz="0 -0.25 0" rpy="0 0 0"/>
     <child link="right_wheel"/>
     <parent link="chassis"/>
@@ -141,5 +141,5 @@
   </link>
   <joint type="fixed" name="camera_joint">
-    <origin xyz="0.2 0 0" rpy="0 0 0"/>
+    <origin xyz="0.2 0 0.1" rpy="0 0 0"/>
     <child link="camera"/>
     <parent link="chassis"/>
@@ -168,5 +168,5 @@
   </link>
   <joint type="fixed" name="hokuyo_joint">
-    <origin xyz="0.15 0 0.1" rpy="0 0 0"/>
+    <origin xyz="0.15 0 0.2" rpy="0 0 0"/>
     <child link="hokuyo"/>
     <parent link="chassis"/>
@@ -176,11 +176,11 @@
   </joint>
 	<gazebo reference="left_wheel">
-    	<material>Gazebo/Green</material>
+    	<material>Gazebo/Blue</material>
 	</gazebo>
     <gazebo reference="right_wheel">
-    	<material>Gazebo/Green</material>
+    	<material>Gazebo/Blue</material>
 	</gazebo>
     <gazebo reference="chassis">
-    	<material>Gazebo/Blue</material>
+    	<material>Gazebo/Black</material>
 	</gazebo>
     <gazebo reference="camera">

Commit message: smaller robot default params

File: catkin_ws/src/my_robot/urdf/my_robot.xacro (robot description, xacro)
@@ -22,5 +22,5 @@
       <origin xyz="0 0 0" rpy=" 0 0 0"/>
       <geometry>
-        <box size=".8 .4 .2"/>
+        <box size=".4 .2 .1"/>
       </geometry>
     </collision>
@@ -28,30 +28,30 @@
       <origin xyz="0 0 0" rpy=" 0 0 0"/>
       <geometry>
-        <box size=".8 .4 .2"/>
+        <box size=".4 .2 .1"/>
       </geometry>
       <material name="black"/>
     </visual>
     <collision name='back_caster_collision'>
-      <origin xyz="-0.15 0 -0.1" rpy=" 0 0 0"/>
+      <origin xyz="-0.15 0 -0.05" rpy=" 0 0 0"/>
       <geometry>
-        <sphere radius="0.099"/>
+        <sphere radius="0.0499"/>
       </geometry>
     </collision>
     <visual name='back_caster_visual'>
-      <origin xyz="-0.15 0 -0.1" rpy=" 0 0 0"/>
+      <origin xyz="-0.15 0 -0.05" rpy=" 0 0 0"/>
       <geometry>
-        <sphere radius="0.1"/>
+        <sphere radius="0.05"/>
       </geometry>
     </visual>
     <collision name='front_caster_collision'>
-      <origin xyz="0.15 0 -0.1" rpy=" 0 0 0"/>
+      <origin xyz="0.15 0 -0.05" rpy=" 0 0 0"/>
       <geometry>
-        <sphere radius="0.099"/>
+        <sphere radius="0.0499"/>
       </geometry>
     </collision>
     <visual name='front_caster_visual'>
-      <origin xyz="0.15 0 -0.1" rpy=" 0 0 0"/>
+      <origin xyz="0.15 0 -0.05" rpy=" 0 0 0"/>
       <geometry>
-        <sphere radius="0.1"/>
+        <sphere radius="0.05"/>
       </geometry>
     </visual>
@@ -66,5 +66,5 @@
       <origin xyz="0 0 0" rpy="0 1.5707 1.5707" />
       <geometry>
-          <cylinder radius='0.2' length='0.05' />
+          <cylinder radius='0.1' length='0.05' />
       </geometry>
     </collision>
@@ -72,5 +72,5 @@
       <origin xyz="0 0 0" rpy="0 1.5707 1.5707" />
       <geometry>
-          <cylinder radius='0.2' length='0.05' />
+          <cylinder radius='0.1' length='0.05' />
       </geometry>
       <material name="blue"/>
@@ -90,5 +90,5 @@
       <origin xyz="0 0 0" rpy="0 1.5707 1.5707" />
       <geometry>
-          <cylinder radius="0.2" length="0.05" />
+          <cylinder radius="0.1" length="0.05" />
       </geometry>
     </collision>
@@ -96,5 +96,5 @@
       <origin xyz="0 0 0" rpy="0 1.5707 1.5707" />
       <geometry>
-          <cylinder radius='0.2' length='0.05' />
+          <cylinder radius='0.1' length='0.05' />
       </geometry>
       <material name="blue"/>
@@ -102,5 +102,5 @@
   </link>
   <joint type="continuous" name="left_wheel_hinge">
-    <origin xyz="0 0.25 0" rpy="0 0 0"/>
+    <origin xyz="0 0.15 0" rpy="0 0 0"/>
     <child link="left_wheel"/>
     <parent link="chassis"/>
@@ -111,5 +111,5 @@
   </joint>
   <joint type="continuous" name="right_wheel_hinge">
-    <origin xyz="0 -0.25 0" rpy="0 0 0"/>
+    <origin xyz="0 -0.15 0" rpy="0 0 0"/>
     <child link="right_wheel"/>
     <parent link="chassis"/>
@@ -141,5 +141,5 @@
   </link>
   <joint type="fixed" name="camera_joint">
-    <origin xyz="0.2 0 0.1" rpy="0 0 0"/>
+    <origin xyz="0.2 0 0" rpy="0 0 0"/>
     <child link="camera"/>
     <parent link="chassis"/>
@@ -168,5 +168,5 @@
   </link>
   <joint type="fixed" name="hokuyo_joint">
-    <origin xyz="0.15 0 0.2" rpy="0 0 0"/>
+    <origin xyz="0.15 0 0.1" rpy="0 0 0"/>
     <child link="hokuyo"/>
     <parent link="chassis"/>
